Commit message: updated orientation of the 6 legged urdf. added readme

File: spiderbot_description/urdf/spiderbot.urdf.xacro (robot description, xacro)
@@ -1,10 +1,12 @@
 <?xml version="1.0"?>
 <robot xmlns:xacro="http://www.ros.org/wiki/xacro" name="spiderbot">
-	<xacro:property name="body_radius" value="0.3"/>
+	<xacro:property name="body_radius" value="0.25"/>
 	<xacro:property name="body_height" value="0.2"/>
 	<xacro:property name="body_mass" value="0.4"/>
-	<xacro:property name="leg_pan_connector_radius" value="0.1"/>
+	<xacro:property name="leg_pan_connector_radius" value="0.08"/>
 	<xacro:property name="leg_pan_connector_height" value="0.05"/>
 	<xacro:property name="leg_pan_vel" value="1.0"/>
+	<xacro:property name="leg_pan_max_angle" value="0.5236"/>
+	<xacro:property name="leg_pan_min_angle" value="-0.5236"/>
 	<xacro:property name="upper_leg_mass" value="0.1"/>
 	<xacro:property name="upper_leg_length" value="0.2"/>
@@ -98,5 +100,5 @@
             <axis xyz="0 0 1"/>
             <origin rpy="0 0 ${yaw}" xyz="${x} ${y} ${z}"/>
-            <limit effort="1000" lower="-0.7854" upper="0.7854" velocity="${leg_pan_vel}"/>
+            <limit effort="1000" lower="${leg_pan_min_angle}" upper="${leg_pan_max_angle}" velocity="${leg_pan_vel}"/>
         </joint>
         <transmission name="leg_${number}_pan_joint_transmission">
@@ -160,10 +162,10 @@
 	-->
 	<!-- 6 leg setup -->
-	<xacro:leg number="1" x="${body_radius}" y="0" z="0" yaw="0"/>
-	<xacro:leg number="2" x="${body_radius*0.5}" y="${-body_radius*0.866}" z="0" yaw="-1.0472"/>
-	<xacro:leg number="3" x="${-body_radius*0.5}" y="${-body_radius*0.866}" z="0" yaw="-2.0944"/>
-	<xacro:leg number="4" x="${-body_radius}" y="0" z="0" yaw="-3.142"/>
-	<xacro:leg number="5" x="${-body_radius*0.5}" y="${body_radius*0.866}" z="0" yaw="2.0944"/>
-	<xacro:leg number="6" x="${body_radius*0.5}" y="${body_radius*0.866}" z="0" yaw="1.0472"/>
+	<xacro:leg number="1" x="${body_radius*0.866}" y="${-body_radius*0.5}" z="0" yaw="-0.5236"/>
+	<xacro:leg number="2" x="0" y="${-body_radius}" z="0" yaw="-1.57075"/>
+	<xacro:leg number="3" x="${-body_radius*0.866}" y="${-body_radius*0.5}" z="0" yaw="-2.6180"/>
+	<xacro:leg number="4" x="${-body_radius*0.866}" y="${body_radius*0.5}" z="0" yaw="2.6180"/>
+	<xacro:leg number="5" x="0" y="${body_radius}" z="0" yaw="1.57075"/>
+	<xacro:leg number="6" x="${body_radius*0.866}" y="${body_radius*0.5}" z="0" yaw="0.5236"/>
 	<gazebo>
         <plugin name="gazebo_ros_control" filename="libgazebo_ros_control.so">
